Commit message: update

File: models/object.urdf.xacro (robot description, xacro)
@@ -1,19 +1,12 @@
 <?xml version="1.0"?>
 <robot
-    xmlns:xacro="http://www.ros.org/wiki/xacro" name="target_location" >
+    xmlns:xacro="http://www.ros.org/wiki/xacro" name="object" >
     <!-- Variables: -->
-    <xacro:property name="position" value="0.5 -0.5 0.05" />
-    <xacro:property name="size" value="0.2 0.2 0.1" />
-    <!-- Used for fixing robot to Gazebo 'world' -->
-    <link name="world" />
-    <joint name="fixed" type="fixed">
-        <parent link="world" />
-        <child link="core" />
-    </joint>
-    <!-- Core: target location object -->
+    <xacro:property name="position" value="0.5 0.0 0.5" />
+    <xacro:property name="size" value="0.02 0.02 0.2" />
     <link name="core">
         <inertial>
-            <origin xyz="0 0 0" />
-            <mass value="1.0" />
+            <origin xyz="${position}" />
+            <mass value="0.01" />
             <inertia ixx="0.0" ixy="0.0" ixz="0.0" iyy="0.0" iyz="0.0" izz="0.0" />
         </inertial>
@@ -33,6 +26,8 @@
     <!-- Gazebo settings -->
     <gazebo reference="core">
-        <gravity>0</gravity>
+        <gravity>1</gravity>
         <material>Gazebo/Red</material>
+        <mu1>130.0</mu1>
+        <mu2>130.0</mu2>
     </gazebo>
 </robot>

File: models/table.urdf.xacro (robot description, xacro)
@@ -1,10 +1,15 @@
 <?xml version="1.0"?>
 <robot
-    xmlns:xacro="http://www.ros.org/wiki/xacro" name="target_object" >
+    xmlns:xacro="http://www.ros.org/wiki/xacro" name="table" >
     <!-- Variables: -->
-    <xacro:property name="position" value="0.5 0.5 0.15" />
-    <xacro:property name="radius" value="0.025" />
-    <xacro:property name="length" value="0.3" />
-    <!-- Core: target location object -->
+    <xacro:property name="position" value="0.0 0.0 0.2" />
+    <xacro:property name="radius" value="0.2" />
+    <xacro:property name="length" value="0.4" />
+    <!-- Used for fixing robot to Gazebo 'world' -->
+    <link name="world" />
+    <joint name="fixed" type="fixed">
+        <parent link="world" />
+        <child link="core" />
+    </joint>
     <link name="core">
         <inertial>
@@ -32,5 +37,5 @@
     <gazebo reference="core">
         <gravity>0</gravity>
-        <material>Gazebo/Orange</material>
+        <material>Gazebo/PaintedWall</material>
     </gazebo>
 </robot>
